File: Main_Board_584/Main_Board_584.sch (KiCad schematic (older format))
At the start: 36 parts

Commit message: Radio and uSD
Finished radio and uSD
Parts:
- removed C?: 100nF, symbol C
- added C? (x2): 100nF, symbol C
- added C?: 10uF, symbol C
- added L?: Ferrite_Bead, symbol Ferrite_Bead_Small
- added U?: ADXL355, symbol ADXL355
- J?: value Conn_Coaxial -> Edge_SMA
Connections:
- net labels added: MISO, MOSI, RADIO_CS, RADIO_INT, RADIO_RST, SCK, SCLK, VDDANA, uSD_CS
- wire segments 96 -> 122
- no-connect marks 3 -> 10
Other:
- moved on the sheet: C?, J?, U?

Commit message: Changes
Parts:
- removed C?: 1uF, symbol C
- removed C?: 470pF, symbol C
- removed C?: 2.2uF, symbol C
- removed C?: 100nF, symbol C
- removed U?: RFM95W, symbol RFM95W
- removed U?: MIC5219-3.3, TO_SOT_Packages_SMD:SOT-23-5, symbol MIC5219-3.3
- added BT?: 18650b, symbol Battery_Cell
- added C? (x4): 100nF, symbol C
- added C? (x3): 0.27uF, symbol C
- added C? (x2): 22uF, symbol C
- added C?: 3.3nF, symbol C
- added D? (x2): LED, symbol LED
- added R? (x2): 330, symbol R
- added R?: 1.21M, symbol R
- added R?: 383K, symbol R
- added U?: RFM23BP, symbol RFM23BP
- added U?: LMZ21701, symbol LMZ21701
Connections:
- net labels added: ACCEL_ST, ACCEL_X, ACCEL_Y, ACCEL_Z, BARO_CS, RADIO_RX, RADIO_TX
- net labels removed: RADIO_RST
- wire segments 122 -> 177
- no-connect marks 10 -> 14
Other:
- note added: "LAYOUT: 1 100nF Per Sensor\n"
- moved on the sheet: D?, R?, U?

Commit message: Changes
Parts:
- removed C? (x3): 0.27uF, symbol C
- removed U?: ADXL355, symbol ADXL355
- added C? (x4): 100nF, symbol C
- added R? (x2): 3.3K, symbol R
- added U?: MPU9250, symbol MPU9250
- added U?: HDC1080, symbol HDC1080
Connections:
- net labels added: MPU_CS, SCL, SDA
- net labels removed: ACCEL_ST, ACCEL_X, ACCEL_Y, ACCEL_Z
- wire segments 177 -> 187
Other:
- note added: "LAYOUT: 1 100nF Per Sensor (MPU gets 2)\n"
- note removed: "LAYOUT: 1 100nF Per Sensor\n"
- moved on the sheet: C?

Commit message: Changes
Parts:
- added C? (x2): 100nF, symbol C
- added U?: TMP36, symbol TMP36
- added U?: UltimateGPS, symbol UltimateGPS
Connections:
- net 3V3: now also C?.1, C?.1, U?.1 (3.3), U?.2 (VS)
- net GND: now also C?.2, C?.2, U?.5 (GND), U?.7 (GND)
- new net RX: U?.5 (TX)
- new net TMP_VOUT: U?.1 (VOUT)
- new net TMP_nSHDN: U?.4 (nSHDN)
- new net TX: U?.6 (RX)
- no-connect marks 14 -> 20
Other:
- note added: "uC Perspective"
- moved on the sheet: C?, J?, R?, U?

Commit message: Changes
Parts:
- added C22, C23: 18pF, Capacitors_SMD:C_0603, symbol C
- added J5, J6: Conn_01x02, MASA:A33199CT-ND, symbol Conn_01x02
- added M1, M2, M3, M4, M5: M3, Mounting_Holes:MountingHole_3.2mm_M3, symbol M3
- added Q1: Q_NJFET_GDS, TO_SOT_Packages_THT:TO-220-3_Vertical, symbol Q_NJFET_GDS
- added R15: 470m, Resistors_THT:R_Axial_DIN0918_L18.0mm_D9.0mm_P25.40mm_Horizontal, symbol R
- added Y1: Crystal, Crystals:Crystal_SMD_EuroQuartz_EQ161-2pin_3.2x1.5mm, symbol Crystal
- BT1, BT2: renamed from BT?; footprint (none) -> MASA:18650Holder
- C1, C10, C12, C13, C14, C15, C16, C17, C18, C19, C2, C20, C21, C3, C4, C5, C6, C7, C9: renamed from C?; footprint (none) -> Capacitors_SMD:C_0603
- C11, C8: renamed from C?; footprint (none) -> Capacitors_SMD:C_1206
- D1, D2, D3, D4, D5, D6, D7: renamed from D?; footprint (none) -> LEDs:LED_0603
- D10, D11, D9: renamed from D?; value D_TVS -> CPDUR5V0HE-HF; footprint (none) -> Diodes_SMD:D_0603
- D8: renamed from D?; value D_Schottky -> B130-13-F; footprint (none) -> Diodes_SMD:D_SMA
- J1: renamed from J?; footprint (none) -> MASA:M50-3600542
- J2: renamed from J?; footprint (none) -> Connectors:USB_Micro-B
- J3: renamed from J?; footprint (none) -> Connectors:microSD_Card_Receptacle_Wuerth_693072010801
- J4: renamed from J?; footprint (none) -> MASA:EBAY_SMA
- L1: renamed from L?; footprint (none) -> Capacitors_SMD:C_0603
- R1, R10, R11, R12, R13, R14, R2, R3, R4, R5, R6, R7, R8, R9: renamed from R?; footprint (none) -> Capacitors_SMD:C_0603
- U1: renamed from U?; footprint (none) -> Housings_DFN_QFN:QFN-48-1EP_7x7mm_Pitch0.5mm
- U2: renamed from U?; footprint (none) -> MASA:LMZ21701
- U3: renamed from U?; footprint (none) -> TO_SOT_Packages_SMD:TSOT-23-5
- U4: renamed from U?; footprint (none) -> MASA:MS5607
- U5: renamed from U?; footprint (none) -> MASA:WSON-6
- U6: renamed from U?; footprint (none) -> MASA:RFM23BP
- U7: renamed from U?; footprint (none) -> Housings_DFN_QFN:QFN-24-1EP_3x3mm_Pitch0.4mm
- U8: renamed from U?; footprint (none) -> MASA:UltimateGPS
Connections:
- net 3V3: now also U7.1 (RESV)
- net GND: now also U1.49 (EP), U7.20 (RESV), C22.2, C23.2, M1.1, M2.1, M3.1, M4.1, M5.1, Q1.3 (S)
- net MOSI: now also U1.25 (PA16); no longer U1.24 (PA15)
- net SCK: now also U1.26 (PA17); no longer U1.25 (PA16)
- net SCL: now also U1.32 (PA23)
- net SDA: now also U1.31 (PA22)
- net VIN: now also J5.2 (Pin_2), J6.2 (Pin_2); no longer BT1.1 (+)
- net nRESET: now also U1.40 (nRESET)
- net at U1.1 (PA00): now also C22.1, Y1.1
- net at U1.2 (PA01): now also C23.1, Y1.2
- new net: J6.1 (Pin_1), R15.2
- new net: Q1.2 (D), R15.1
- new net FTU_FIRE: Q1.1 (G)
- new net VBAT: BT1.1 (+), J5.1 (Pin_1)
- no-connect marks 20 -> 19
Other:
- note added: "Nichrome\n"
- note added: "Power\nSwitch\n"

Commit message: Fixes
Fixed some things
Connections:
- net GND: now also U7.11 (FSYNC)
- net MISO: now also U7.9 (SDO); no longer U7.24 (SDI)
- net MOSI: now also U7.24 (SDI); no longer U7.9 (SDO)
- no-connect marks 19 -> 18
Changed lines of the file:
@@
 $EndComp
 Text Label 13050 3500 0    60   ~ 0
+MISO
+Text Label 13050 3600 0    60   ~ 0
 MOSI
-Text Label 13050 3600 0    60   ~ 0
-MISO
 Text Label 13050 3700 0    60   ~ 0
 SCLK
 Text Label 13050 3800 0    60   ~ 0
 MPU_CS
-NoConn ~ 13450 3350
 Text GLabel 14700 3800 2    60   Input ~ 0
 GND
@@
 	12700 3250 12700 3300
 Wire Wire Line
-	12400 3650 12700 3650
+	12400 3650 12800 3650
 Wire Wire Line
 	12700 3650 12700 3600
@@
 Text GLabel 2300 6750 2    60   Input ~ 0
 GND
+Wire Wire Line
+	13450 3350 12800 3350
+Wire Wire Line
+	12800 3350 12800 3650
+Connection ~ 12700 3650
 $EndSCHEMATC

Commit message: Board Changes
Connections:
- net SCK is gone; now on net SCLK: U1.26 (PA17), U6.4 (SCK)
Changed lines of the file:
@@
 GND
 Text Label 4400 4050 0    60   ~ 0
-SCK
+SCLK
 Text Label 4400 3950 0    60   ~ 0
 MOSI
@@
 MOSI
 Text Label 12800 1550 0    60   ~ 0
-SCK
+SCLK
 Text Label 12800 1650 0    60   ~ 0
 RADIO_CS

Commit message: added thermistor circuit
Parts:
- added C25: 100nF, Capacitors_SMD:C_0603, symbol C
- added J7: Conn_01x02, MASA:A33199CT-ND, symbol Conn_01x02
- added R14: 100k 1%, Capacitors_SMD:C_0603, symbol R
- added U?: MCP6001T-I_OT, digikey-footprints:SOT-753, symbol MCP6001T-I_OT
Connections:
- net GND: now also C25.2, J7.2 (Pin_2), U?.2 (VSS)
- new net: J7.1 (Pin_1), U?.3 (VIN+)
- new net 2V5: C25.1, R14.2, U?.5 (VDD)
- new net THERM: U?.1 (VOUT), U?.4 (VIN-)
Other:
- note added: "Thermistor"
