File: Main_Board_584/Main_Board_584.sch (KiCad schematic (older format))
At the start: 107 parts, among them J1 Conn_02x05_Top_Bottom, J10 Conn_01x02, J2 USB_OTG, J3 Micro_SD_Card, J4 Edge_SMA, J5 Conn_01x02, J6 Conn_01x02, J7 Conn_01x02, J8 Conn_01x02, J9 Conn_01x02, M1 M3, M2 M3, M3 M3, M4 M3, M5 M3, Q1 Q_NJFET_GDS, Q2 Q_NJFET_GDS, U1 SAMD21G18A, U10 LT1461, U2 LMZ21701, U3 TMP36, U4 MS5607, U5 HDC1080, U6 RFM23BP, U7 MPU9250, U8 UltimateGPS, U9 MCP6001T-I_OT, Y1 Crystal

Commit message: Mid Board Design
Parts:
- removed C6: 100nF, Capacitors_SMD:C_0603, symbol C
- removed C7: 10uF, Capacitors_SMD:C_0603, symbol C
- removed L1: Ferrite_Bead, Capacitors_SMD:C_0603, symbol Ferrite_Bead_Small
- removed TP19: TEST, MASA:0603_TP, symbol TEST
- added R20, R21: 330, Capacitors_SMD:C_0603, symbol R
- added TP21, TP22, TP23: TEST, MASA:0603_TP, symbol TEST
- U9: footprint digikey-footprints:SOT-753 -> TO_SOT_Packages_SMD:SOT-23-5
Connections:
- net VDDANA is gone; now on net 2V5: U1.6 (VDDANA)
- net 3V3: now also TP22.1
- net GND: now also R21.1, TP21.1, TP23.1; no longer TP20.1
- net VBAT: now also R20.2
- net at J7.1 (Pin_1), R19.1, U9.3 (VIN+): now also TP20.1
- new net BAT_SENSE: R20.1, R21.2
Other:
- moved on the sheet: TP20
Changed lines of the file:
@@
 Text Notes 9150 8800 0    60   ~ 0
 Move diode depending on if USB or Batt voltage is higher\n
-Text GLabel 6000 6650 2    60   Input ~ 0
+Text GLabel 6300 6650 2    60   Input ~ 0
 VBAT
-Text GLabel 5550 7450 2    60   Input ~ 0
+Text GLabel 6300 7450 2    60   Input ~ 0
 GND
 $Comp
@@
 Text Label 12800 1650 0    60   ~ 0
 RADIO_CS
-$Comp
-L Ferrite_Bead_Small L1
-U 1 1 5A5EBD3C
-P 2350 1550
-F 0 "L1" V 2400 1650 50  0000 L CNN
-F 1 "Ferrite_Bead" V 2200 1350 50  0000 L CNN
-F 2 "Capacitors_SMD:C_0603" V 2280 1550 50  0001 C CNN
-F 3 "" H 2350 1550 50  0001 C CNN
-	1    2350 1550
-	0    1    1    0
-$EndComp
-Text Label 3500 1550 2    60   ~ 0
-VDDANA
-$Comp
-L C C6
-U 1 1 5A5EC299
-P 2600 1750
-F 0 "C6" H 2625 1850 50  0000 L CNN
-F 1 "100nF" H 2625 1650 50  0000 L CNN
-F 2 "Capacitors_SMD:C_0603" H 2638 1600 50  0001 C CNN
-F 3 "" H 2600 1750 50  0001 C CNN
-	1    2600 1750
-	1    0    0    -1
-$EndComp
-$Comp
-L C C7
-U 1 1 5A5EC34E
-P 2950 1750
-F 0 "C7" H 2975 1850 50  0000 L CNN
-F 1 "10uF" H 2975 1650 50  0000 L CNN
-F 2 "Capacitors_SMD:C_0603" H 2988 1600 50  0001 C CNN
-F 3 "" H 2950 1750 50  0001 C CNN
-	1    2950 1750
-	1    0    0    -1
-$EndComp
-Text GLabel 4350 1650 0    60   Input ~ 0
+Text GLabel 4350 1650 0    55   Input ~ 0
 3V3
-Text Label 4400 1550 0    60   ~ 0
-VDDANA
 NoConn ~ 9600 1300
 Text Label 9100 1400 0    60   ~ 0
@@
 F 0 "U9" H 14400 8450 60  0000 C CNN
 F 1 "MCP6001T-I_OT" H 14600 8650 60  0000 C CNN
-F 2 "digikey-footprints:SOT-753" H 14800 8350 60  0001 L CNN
+F 2 "TO_SOT_Packages_SMD:SOT-23-5" H 14800 8350 60  0001 L CNN
 F 3 "http://www.microchip.com/mymicrochip/filehandler.aspx?ddocname=en011705" H 14800 8450 60  0001 L CNN
 F 4 "MCP6001T-I/OTCT-ND" H 14800 8550 60  0001 L CNN "Digi-Key_PN"
@@
 	4800 1950 4400 1950
 Wire Wire Line
-	1100 1900 1100 1950
+	1100 1950 1100 1900
 Wire Wire Line
 	1400 1950 1400 1900
@@
 	5400 7350 5400 7450
 Wire Wire Line
-	5400 7450 5550 7450
+	5400 7450 6300 7450
 Wire Wire Line
 	8500 9850 8800 9850
@@
 Wire Wire Line
 	12800 1650 13400 1650
-Wire Wire Line
-	950  1950 2950 1950
 Connection ~ 1750 1950
 Connection ~ 1400 1950
 Connection ~ 1100 1950
-Wire Wire Line
-	950  1550 2250 1550
 Connection ~ 1750 1550
 Connection ~ 1400 1550
 Connection ~ 1100 1550
 Connection ~ 2100 1550
-Wire Wire Line
-	2450 1550 3500 1550
-Wire Wire Line
-	2950 1950 2950 1900
 Connection ~ 2100 1950
 Wire Wire Line
-	2600 1900 2600 1950
-Connection ~ 2600 1950
-Wire Wire Line
-	2600 1600 2600 1550
-Connection ~ 2600 1550
-Wire Wire Line
-	2950 1600 2950 1550
-Connection ~ 2950 1550
-Wire Wire Line
 	4700 1650 4700 1850
 Wire Wire Line
-	4800 1550 4400 1550
+	4350 1550 4800 1550
 Wire Wire Line
 	9600 1400 9100 1400
@@
 Connection ~ 14600 3700
 Wire Wire Line
-	5400 6650 6000 6650
+	5400 6650 6300 6650
 Wire Wire Line
 	2550 5500 2400 5500
@@
 	14050 8250 14050 8150
 Connection ~ 14050 8150
-Connection ~ 15450 7500
-Wire Wire Line
-	15400 8550 15450 8550
-Connection ~ 15450 8550
-Wire Wire Line
-	15400 7500 15450 7500
 $Comp
 L TEST TP6
@@
 $EndComp
 $Comp
-L TEST TP19
-U 1 1 5A71433D
-P 15400 7500
-F 0 "TP19" H 15400 7700 50  0000 C BNN
-F 1 "TEST" H 15400 7750 50  0001 C CNN
-F 2 "MASA:0603_TP" H 15400 7500 50  0001 C CNN
-F 3 "" H 15400 7500 50  0001 C CNN
-	1    15400 7500
-	0    -1   -1   0
-$EndComp
-$Comp
 L TEST TP20
 U 1 1 5A7145C8
-P 15400 8550
-F 0 "TP20" H 15400 8750 50  0000 C BNN
-F 1 "TEST" H 15400 8800 50  0001 C CNN
-F 2 "MASA:0603_TP" H 15400 8550 50  0001 C CNN
-F 3 "" H 15400 8550 50  0001 C CNN
-	1    15400 8550
+P 15200 8450
+F 0 "TP20" H 15200 8650 50  0000 C BNN
+F 1 "TEST" H 15200 8700 50  0001 C CNN
+F 2 "MASA:0603_TP" H 15200 8450 50  0001 C CNN
+F 3 "" H 15200 8450 50  0001 C CNN
+	1    15200 8450
 	0    -1   -1   0
 $EndComp
@@
 Wire Wire Line
 	2100 6500 2550 6500
+$Comp
+L TEST TP22
+U 1 1 5A755234
+P 7200 9300
+F 0 "TP22" H 7200 9500 50  0000 C BNN
+F 1 "TEST" H 7200 9550 50  0001 C CNN
+F 2 "MASA:0603_TP" H 7200 9300 50  0001 C CNN
+F 3 "" H 7200 9300 50  0001 C CNN
+	1    7200 9300
+	1    0    0    -1
+$EndComp
+Wire Wire Line
+	7200 9350 7200 9300
+Connection ~ 7200 9350
+$Comp
+L TEST TP23
+U 1 1 5A7555C5
+P 7200 10000
+F 0 "TP23" H 7200 10200 50  0000 C BNN
+F 1 "TEST" H 7200 10250 50  0001 C CNN
+F 2 "MASA:0603_TP" H 7200 10000 50  0001 C CNN
+F 3 "" H 7200 10000 50  0001 C CNN
+	1    7200 10000
+	1    0    0    -1
+$EndComp
+Wire Wire Line
+	7200 10100 7200 10000
+Connection ~ 7200 10100
+$Comp
+L TEST TP21
+U 1 1 5A755930
+P 7050 10000
+F 0 "TP21" H 7050 10200 50  0000 C BNN
+F 1 "TEST" H 7050 10250 50  0001 C CNN
+F 2 "MASA:0603_TP" H 7050 10000 50  0001 C CNN
+F 3 "" H 7050 10000 50  0001 C CNN
+	1    7050 10000
+	1    0    0    -1
+$EndComp
+Wire Wire Line
+	7050 10100 7050 10000
+Connection ~ 7050 10100
+$Comp
+L R R20
+U 1 1 5A75891F
+P 6100 6850
+F 0 "R20" V 6180 6850 50  0000 C CNN
+F 1 "330" V 6100 6850 50  0000 C CNN
+F 2 "Capacitors_SMD:C_0603" V 6030 6850 50  0001 C CNN
+F 3 "" H 6100 6850 50  0001 C CNN
+	1    6100 6850
+	-1   0    0    1
+$EndComp
+$Comp
+L R R21
+U 1 1 5A758C37
+P 6100 7250
+F 0 "R21" V 6180 7250 50  0000 C CNN
+F 1 "330" V 6100 7250 50  0000 C CNN
+F 2 "Capacitors_SMD:C_0603" V 6030 7250 50  0001 C CNN
+F 3 "" H 6100 7250 50  0001 C CNN
+	1    6100 7250
+	-1   0    0    1
+$EndComp
+Wire Wire Line
+	6100 6650 6100 6700
+Connection ~ 6100 6650
+Wire Wire Line
+	6100 7100 6100 7000
+Wire Wire Line
+	6100 7050 6700 7050
+Connection ~ 6100 7050
+Text Label 6700 7050 2    60   ~ 0
+BAT_SENSE
+Wire Wire Line
+	6100 7450 6100 7400
+Connection ~ 6100 7450
+Wire Wire Line
+	15200 8450 15300 8450
+Wire Wire Line
+	15300 8450 15300 8250
+Connection ~ 15300 8250
+Wire Wire Line
+	950  1950 2100 1950
+Wire Wire Line
+	950  1550 2100 1550
+Text GLabel 4350 1550 0    55   Input ~ 0
+2V5
 $EndSCHEMATC

Commit message: Board Done
Parts:
- M1, M2, M3, M4, M5: footprint Mounting_Holes:MountingHole_3.2mm_M3 -> MASA:M3Mounting_Hole
Connections:
- net 3V3: now also C24.1, TP3.1, U10.2 (VIN), U10.3 (nSHDN)
- net AIN_1: now also U1.13 (PA08)
- net AIN_2: now also U1.15 (PA10)
- net BARO_CS: now also U1.47 (PB02)
- net BAT_SENSE: now also U1.14 (PA09)
- net FTU_FIRE: now also U1.22 (PA13)
- net HEAT_ON: now also U1.23 (PA14)
- net HOST_EN: now also U1.39 (PA27); no longer U1.41 (PA28)
- net LED_1: now also U1.7 (PB08)
- net LED_2: now also U1.8 (PB09)
- net LED_3: now also U1.9 (PA04)
- net LED_4: now also U1.10 (PA05)
- net MPU_CS: now also U1.41 (PA28)
- net RADIO_CS: now also U1.48 (PB03)
- net RX: now also U1.38 (PB23)
- net THERM: now also U1.16 (PA11)
- net TMP_VOUT: now also U1.11 (PA06)
- net TMP_nSHDN: now also U1.12 (PA07)
- net TX: now also U1.37 (PB22)
- net VIN: no longer C24.1, TP3.1, U10.2 (VIN), U10.3 (nSHDN)
- net uSD_CS: now also U1.24 (PA15)
- no-connect marks 18 -> 19
Changed lines of the file:
@@
 GND
 Text Label 6550 2450 2    60   ~ 0
-HOST_EN
+MPU_CS
 $Comp
 L Battery_Cell BT2
@@
 F 0 "M1" H 11450 9300 60  0000 C CNN
 F 1 "M3" H 11300 9200 60  0000 C CNN
-F 2 "Mounting_Holes:MountingHole_3.2mm_M3" H 11450 9200 60  0001 C CNN
+F 2 "MASA:M3Mounting_Hole" H 11450 9200 60  0001 C CNN
 F 3 "" H 11450 9200 60  0001 C CNN
 	1    11450 9200
@@
 F 0 "M2" H 11450 9500 60  0000 C CNN
 F 1 "M3" H 11300 9400 60  0000 C CNN
-F 2 "Mounting_Holes:MountingHole_3.2mm_M3" H 11450 9400 60  0001 C CNN
+F 2 "MASA:M3Mounting_Hole" H 11450 9400 60  0001 C CNN
 F 3 "" H 11450 9400 60  0001 C CNN
 	1    11450 9400
@@
 F 0 "M3" H 11450 9700 60  0000 C CNN
 F 1 "M3" H 11300 9600 60  0000 C CNN
-F 2 "Mounting_Holes:MountingHole_3.2mm_M3" H 11450 9600 60  0001 C CNN
+F 2 "MASA:M3Mounting_Hole" H 11450 9600 60  0001 C CNN
 F 3 "" H 11450 9600 60  0001 C CNN
 	1    11450 9600
@@
 F 0 "M4" H 11450 9900 60  0000 C CNN
 F 1 "M3" H 11300 9800 60  0000 C CNN
-F 2 "Mounting_Holes:MountingHole_3.2mm_M3" H 11450 9800 60  0001 C CNN
+F 2 "MASA:M3Mounting_Hole" H 11450 9800 60  0001 C CNN
 F 3 "" H 11450 9800 60  0001 C CNN
 	1    11450 9800
@@
 F 0 "M5" H 11450 10100 60  0000 C CNN
 F 1 "M3" H 11300 10000 60  0000 C CNN
-F 2 "Mounting_Holes:MountingHole_3.2mm_M3" H 11450 10000 60  0001 C CNN
+F 2 "MASA:M3Mounting_Hole" H 11450 10000 60  0001 C CNN
 F 3 "" H 11450 10000 60  0001 C CNN
 	1    11450 10000
@@
 $EndComp
 Text GLabel 8500 7600 0    60   Input ~ 0
-VIN
+3V3
 $Comp
 L C C24
@@
 Text GLabel 4350 1550 0    55   Input ~ 0
 2V5
+Wire Wire Line
+	4800 3650 4400 3650
+Wire Wire Line
+	4800 3750 4400 3750
+Text Label 4400 3750 0    60   ~ 0
+HEAT_ON
+Text Label 4400 3650 0    60   ~ 0
+FTU_FIRE
+Wire Wire Line
+	6100 3000 6550 3000
+Text Label 6550 3000 2    60   ~ 0
+LED_1
+Wire Wire Line
+	4300 2750 4800 2750
+Wire Wire Line
+	4300 2850 4800 2850
+Text Label 6550 3100 2    60   ~ 0
+LED_2
+Text Label 4300 2750 0    60   ~ 0
+LED_3
+Text Label 4300 2850 0    60   ~ 0
+LED_4
+Wire Wire Line
+	4300 2950 4800 2950
+Text Label 4300 2950 0    60   ~ 0
+TMP_VOUT
+Wire Wire Line
+	4800 3050 4300 3050
+Text Label 4300 3050 0    60   ~ 0
+TMP_nSHDN
+Wire Wire Line
+	6550 3100 6100 3100
+Wire Wire Line
+	4800 3150 4300 3150
+Wire Wire Line
+	4300 3250 4800 3250
+Wire Wire Line
+	4800 3350 4300 3350
+Wire Wire Line
+	4300 3450 4800 3450
+Text Label 4300 3150 0    60   ~ 0
+AIN_1
+Text Label 4300 3250 0    60   ~ 0
+BAT_SENSE
+Text Label 4300 3350 0    60   ~ 0
+AIN_2
+Text Label 4300 3450 0    60   ~ 0
+THERM
+Wire Wire Line
+	4800 3850 4400 3850
+Text Label 4400 3850 0    60   ~ 0
+uSD_CS
+Wire Wire Line
+	6100 2350 6550 2350
+Text Label 6550 2350 2    60   ~ 0
+HOST_EN
+Wire Wire Line
+	6100 3400 6550 3400
+Wire Wire Line
+	6550 3500 6100 3500
+Text Label 6550 3500 2    60   ~ 0
+RX
+Text Label 6550 3400 2    60   ~ 0
+TX
+Wire Wire Line
+	6550 2900 6100 2900
+Wire Wire Line
+	6550 2800 6100 2800
+Text Label 6550 2800 2    60   ~ 0
+BARO_CS
+Text Label 6550 2900 2    60   ~ 0
+RADIO_CS
+NoConn ~ 5850 4550
 $EndSCHEMATC

Commit message: Board Done
Connections:
- net RADIO_INT: now also U1.4 (PA03)
- no-connect marks 19 -> 26
Changed lines of the file:
@@
 RADIO_CS
 NoConn ~ 5850 4550
+Wire Wire Line
+	4800 2650 4300 2650
+Text Label 4300 2650 0    60   ~ 0
+RADIO_INT
+NoConn ~ 4800 2550
+NoConn ~ 4800 3550
+NoConn ~ 6100 3300
+NoConn ~ 6100 3200
+NoConn ~ 6100 1850
+NoConn ~ 6100 1750
+NoConn ~ 6100 1650
 $EndSCHEMATC

Commit message: Changes
Parts:
- removed D4, D5: LED, LEDs:LED_0603, symbol LED
- removed R11: 330, Capacitors_SMD:C_0603, symbol R
- added J11, J12: Conn_01x02, MASA:A33199CT-ND, symbol Conn_01x02
- added SW1: SW_Push, Buttons_Switches_SMD:SW_SPST_B3U-1100P, symbol SW_Push
- J1: value Conn_02x05_Top_Bottom -> Conn_02x05
- R20: value 330 -> 20k
- R21: value 330 -> 10k
Connections:
- net BAT_SENSE: now also U1.8 (PB09); no longer U1.14 (PA09)
- net GND: now also SW1.1; no longer J8.1 (Pin_1)
- net LED_1: now also U1.29 (PA20); no longer U1.7 (PB08)
- net LED_2: now also U1.30 (PA21); no longer U1.8 (PB09)
- net LED_3: now also U1.28 (PA19), J11.1 (Pin_1); no longer U1.9 (PA04)
- net LED_4: now also U1.27 (PA18), J12.1 (Pin_1); no longer U1.10 (PA05)
- net MISO: now also U1.21 (PA12); no longer U1.27 (PA18)
- net MOSI: now also U1.19 (PB10); no longer U1.25 (PA16)
- net RADIO_INT: now also U1.3 (PA02); no longer U1.4 (PA03)
- net SCLK: now also U1.20 (PB11); no longer U1.26 (PA17)
- net THERM: now also U1.9 (PA04); no longer U1.16 (PA11)
- net TMP_VOUT: now also U1.7 (PB08); no longer U1.11 (PA06)
- net VIN: now also J9.2 (Pin_2)
- net nRESET: now also SW1.2
- net at R4.2: now also J11.2 (Pin_2)
- net at R5.2: now also J12.2 (Pin_2)
- net AIN_1: no longer names the net of U1.13 (PA08)
- net AIN_1: no longer J8.2 (Pin_2)
- net AIN_2 renamed RX2
- net RX2: now also J8.2 (Pin_2); no longer J9.2 (Pin_2)
- new net TX2: J8.1 (Pin_1), U1.16 (PA11)
- no-connect marks 26 -> 25
Other:
- note added: "External LEDs"
- moved on the sheet: D2, D3, R12, R2, R3, R4, R5
