File: Main_Board_584/Main_Board_584.sch (KiCad schematic (older format))
At the start: 108 parts, among them J1 Conn_02x05, J10 Conn_01x02, J11 Conn_01x02, J12 Conn_01x02, J2 USB_OTG, J3 Micro_SD_Card, J4 Edge_SMA, J5 Conn_01x02, J6 Conn_01x02, J7 Conn_01x02, J8 Conn_01x02, J9 Conn_01x02, M1 M3, M2 M3, M3 M3, M4 M3, M5 M3, Q1 Q_NJFET_GDS, Q2 Q_NJFET_GDS, SW1 SW_Push, U1 SAMD21G18A, U10 LT1461, U2 LMZ21701, U3 TMP36, U4 MS5607, U5 HDC1080, U6 RFM23BP, U7 MPU9250, U8 UltimateGPS, U9 MCP6001T-I_OT, Y1 Crystal

Commit message: Fixed Stuff
Parts:
- added TP19, TP24: TEST, MASA:0603_TP, symbol TEST
Connections:
- net HOST_EN is gone; now on net RADIO_CS: U1.39 (PA27)
- net 3V3: now also J1.1 (Pin_1); no longer J1.6 (Pin_6)
- net GND: now also J1.2 (Pin_2), J1.3 (Pin_3), J1.5 (Pin_5); no longer J1.10 (Pin_10), J1.7 (Pin_7), J1.8 (Pin_8)
- net RADIO_CS: no longer U1.48 (PB03)
- net SWCLK: now also J1.7 (Pin_7); no longer J1.2 (Pin_2)
- net SWDIO: now also J1.6 (Pin_6); no longer J1.1 (Pin_1)
- net nRESET: now also J1.10 (Pin_10); no longer J1.5 (Pin_5)
- net at U1.25 (PA16): now also TP19.1
- net at U1.26 (PA17): now also TP24.1
- no-connect marks 25 -> 24
Changed lines of the file:
@@
 L Conn_02x05_Top_Bottom J1
 U 1 1 5A5A7249
-P 6050 8200
-F 0 "J1" H 6100 8500 50  0000 C CNN
-F 1 "Conn_02x05" H 6100 7900 50  0000 C CNN
-F 2 "MASA:M50-3600542" H 6050 8200 50  0001 C CNN
-F 3 "" H 6050 8200 50  0001 C CNN
-	1    6050 8200
-	1    0    0    -1
+P 6150 8200
+F 0 "J1" H 6200 8500 50  0000 C CNN
+F 1 "Conn_02x05" H 6200 7900 50  0000 C CNN
+F 2 "MASA:M50-3600542" H 6150 8200 50  0001 C CNN
+F 3 "" H 6150 8200 50  0001 C CNN
+	1    6150 8200
+	-1   0    0    -1
 $EndComp
 NoConn ~ 5850 8200
@@
 uSD_CS
 Text Label 6600 2350 2    60   ~ 0
-HOST_EN
+RADIO_CS
 Text Label 6600 3500 2    60   ~ 0
 RX
@@
 Text Label 6600 2800 2    60   ~ 0
 BARO_CS
-Text Label 6600 2900 2    60   ~ 0
-RADIO_CS
 Text Label 4300 2550 0    60   ~ 0
 RADIO_INT
@@
 	6100 2800 6600 2800
 Wire Wire Line
-	6100 2900 6600 2900
-Wire Wire Line
 	6100 3500 6600 3500
 Wire Wire Line
@@
 NoConn ~ 4800 2850
 NoConn ~ 4800 2650
-NoConn ~ 4800 3950
-NoConn ~ 4800 4050
+NoConn ~ 6100 2900
+Wire Wire Line
+	4800 3950 4300 3950
+$Comp
+L TEST TP19
+U 1 1 5A746856
+P 4300 4200
+F 0 "TP19" H 4300 4400 50  0000 C BNN
+F 1 "TEST" H 4300 4450 50  0001 C CNN
+F 2 "MASA:0603_TP" H 4300 4200 50  0001 C CNN
+F 3 "" H 4300 4200 50  0001 C CNN
+	1    4300 4200
+	-1   0    0    1
+$EndComp
+$Comp
+L TEST TP24
+U 1 1 5A747192
+P 4500 4200
+F 0 "TP24" H 4500 4400 50  0000 C BNN
+F 1 "TEST" H 4500 4450 50  0001 C CNN
+F 2 "MASA:0603_TP" H 4500 4200 50  0001 C CNN
+F 3 "" H 4500 4200 50  0001 C CNN
+	1    4500 4200
+	-1   0    0    1
+$EndComp
+Wire Wire Line
+	4300 3950 4300 4200
+Wire Wire Line
+	4500 4200 4500 4050
+Wire Wire Line
+	4500 4050 4800 4050
 $EndSCHEMATC
