File: Main_Board_584/Main_Board_584.kicad_pcb (KiCad board)
At the start: 2 copper layers, 100 x 100 mm, 73 parts, among them J1 Conn_02x05_Top_Bottom, J2 USB_OTG, J3 Micro_SD_Card, J4 Edge_SMA, J5 Conn_01x02, J6 Conn_01x02, M1 M3, M2 M3, M3 M3, M4 M3, M5 M3, Q1 Q_NJFET_GDS, U1 SAMD21G18A, U2 LMZ21701, U3 TMP36, U4 MS5607, U5 HDC1080, U6 RFM23BP, U7 MPU9250, U8 UltimateGPS, Y1 Crystal

Commit message: Board Changes
Connections:
- U1 pad 26: /SCK -> /SCLK
- U6 pad 4: /SCK -> /SCLK
- U7 pad 11: Net-(U7-Pad11) -> GND
- U7 pad 24: /MISO -> /MOSI
- U7 pad 9: /MOSI -> /MISO
Routing:
- net /MOSI: track 0.00 -> 136.9 mm, vias 0 -> 5
- net /SCLK: track 0.00 -> 128.5 mm, vias 0 -> 5
- net /MISO: track 0.00 -> 125.2 mm, vias 0 -> 5
- net GND: track 0.00 -> 85.5 mm, vias 0 -> 57
- net VIN: track 0.00 -> 45.5 mm
- net /USB_N: track 0.00 -> 29.7 mm
- net VBAT: track 0.00 -> 29.6 mm
- net /USB_P: track 0.00 -> 29.5 mm
- net /nRESET: track 0.00 -> 23.3 mm
- net Net-(BT1-Pad2): track 0.00 -> 23.0 mm
- net /SCL: track 0.00 -> 16.4 mm
- net /SWCLK: track 0.00 -> 15.0 mm
- net /SDA: track 0.00 -> 14.7 mm
- net /SWDIO: track 0.00 -> 13.9 mm
- net Net-(J6-Pad1): track 0.00 -> 13.4 mm
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Other:
- copper layers 2 -> 4
- net class Default: trace_width 0.25 -> 0.18; via_dia 0.6 -> 0.65; via_drill 0.4 -> 0.3
- rule trace_min: 0.2 -> 0.16

Commit message: Mid Board Design
Parts:
- removed C6: 100nF, Capacitors_SMD:C_0603
- removed C7: 10uF, Capacitors_SMD:C_0603
- removed L1: Ferrite_Bead, Capacitors_SMD:C_0603
- added C24: 1uF, Capacitors_SMD:C_0603, F.Cu at (163.1, 112.8)
- added C25: 100nF, Capacitors_SMD:C_0603, F.Cu at (157.9, 128.5)
- added C26: 2.2uF, Capacitors_SMD:C_0603, F.Cu at (173.1, 111.4)
- added J10: Conn_01x02, MASA:A33199CT-ND, F.Cu at (117.0, 144.5)
- added J7: Conn_01x02, MASA:A33199CT-ND, F.Cu at (152.7, 134.7)
- added J8: Conn_01x02, MASA:A33199CT-ND, F.Cu at (158.3, 107.2)
- added J9: Conn_01x02, MASA:A33199CT-ND, F.Cu at (158.3, 121.8)
- added Q2: Q_NJFET_GDS, TO_SOT_Packages_THT:TO-220-3_Vertical, F.Cu at (105.1, 139.6)
- added R16: 330, Capacitors_SMD:C_0603, F.Cu at (163.8, 124.4)
- added R17: 0, Capacitors_SMD:C_0603, F.Cu at (155.6, 90.4)
- added R18: 0, Capacitors_SMD:C_0603, F.Cu at (158.2, 90.4)
- added R19: 100k 1%, Capacitors_SMD:C_0603, F.Cu at (147.7, 133.7)
- added R20: 330, Capacitors_SMD:C_0603, F.Cu at (161.4, 118.8)
- added R21: 330, Capacitors_SMD:C_0603, F.Cu at (161.4, 115.8)
- added TP1: TEST, MASA:0603_TP, F.Cu at (159.3, 166.6)
- added TP10: TEST, MASA:0603_TP, F.Cu at (158.6, 126.8)
- added TP11: TEST, MASA:0603_TP, F.Cu at (178.9, 131.3)
- added TP12: TEST, MASA:0603_TP, F.Cu at (178.9, 135.7)
- added TP13: TEST, MASA:0603_TP, F.Cu at (178.9, 133.6)
- added TP14: TEST, MASA:0603_TP, F.Cu at (165.1, 171.6)
- added TP15: TEST, MASA:0603_TP, F.Cu at (158.2, 84.3)
- added TP16: TEST, MASA:0603_TP, F.Cu at (165.3, 167.7)
- added TP17: TEST, MASA:0603_TP, F.Cu at (158.2, 86.7)
- added TP18: TEST, MASA:0603_TP, F.Cu at (160.6, 132.5)
- added TP19: TEST, MASA:0603_TP, F.Cu at (172.6, 177.5)
- added TP2: TEST, MASA:0603_TP, F.Cu at (168.2, 169.8)
- added TP20: TEST, MASA:0603_TP, F.Cu at (153.6, 175.3)
- added TP21: TEST, MASA:0603_TP, F.Cu at (193.3, 97.8)
- added TP22: TEST, MASA:0603_TP, F.Cu at (174.6, 137.6)
- added TP23: TEST, MASA:0603_TP, F.Cu at (164.2, 147.8)
- added TP3: TEST, MASA:0603_TP, F.Cu at (166.6, 147.8)
- added TP4: TEST, MASA:0603_TP, F.Cu at (168.7, 167.8)
- added TP5: TEST, MASA:0603_TP, F.Cu at (169.3, 129.7)
- added TP6: TEST, MASA:0603_TP, F.Cu at (174.6, 168.8)
- added TP7: TEST, MASA:0603_TP, F.Cu at (169.3, 131.6)
- added TP8: TEST, MASA:0603_TP, F.Cu at (174.3, 170.9)
- added TP9: TEST, MASA:0603_TP, F.Cu at (168.5, 174.4)
- added U10: LT1461, Housings_SOIC:SOIC-8_3.9x4.9mm_Pitch1.27mm, F.Cu at (168.2, 111.5)
- added U9: MCP6001T-I_OT, TO_SOT_Packages_SMD:SOT-23-5, F.Cu at (157.7, 131.5)
- moved C21 101.5 mm to (180.1, 98.9), turned to 180 degrees
- moved U3 13.3 mm to (169.8, 104.6)
- moved C14 13.3 mm to (173.5, 103.7)
Connections:
- Q1 pad 1: /FTU_FIRE -> Net-(Q1-Pad1)
- U8 pad 5: /RX -> Net-(R17-Pad2)
- U8 pad 6: /TX -> Net-(R18-Pad2)
Routing:
- net VIN: track 45.5 -> 68.9 mm
- net Net-(J10-Pad1): track 0.00 -> 15.8 mm
- net Net-(R17-Pad2): track 0.00 -> 10.7 mm
- net /VDDANA: track 7.20 -> 0.00 mm
- net Net-(R18-Pad2): track 0.00 -> 6.68 mm
- net /SDA: track 14.7 -> 16.6 mm
- net VBAT: track 29.6 -> 31.4 mm
- net /SCL: track 16.4 -> 17.5 mm
- net GND: track 85.5 -> 86.4 mm, vias 57 -> 60
- net /MISO: track 125.2 -> 125.9 mm, vias 5 -> 6
- net /SCLK: track 128.5 -> 129.0 mm, vias 5 -> 6
- net /MOSI: vias 5 -> 6
Other:
- board text added: "HEAT"

Commit message: Board Done
Parts:
- removed TP19: TEST, MASA:0603_TP
- M1, M2, M3, M4, M5: footprint Mounting_Holes:MountingHole_3.2mm_M3 -> MASA:M3Mounting_Hole
- moved TP14 72.9 mm to (176.2, 99.5), turned to 90 degrees
- moved TP8 67.8 mm to (165.5, 103.7)
- moved TP6 61.3 mm to (169.3, 107.7)
- moved TP9 61.2 mm to (187.3, 116.2)
- moved TP16 53.9 mm to (188.0, 118.8)
- moved TP2 46.0 mm to (167.2, 123.8)
- moved TP1 44.0 mm to (163.6, 122.8)
- moved TP20 42.9 mm to (153.9, 132.4)
- moved TP4 40.7 mm to (169.0, 127.1), turned to 90 degrees
- moved J7 1.00 mm to (152.7, 135.7)
Connections:
- C24 pad 1: VIN -> 3V3
- TP20 pad 1: GND -> Net-(J7-Pad1)
- TP3 pad 1: VIN -> 3V3
- U1 pad 10: Net-(U1-Pad10) -> /LED_4
- U1 pad 11: Net-(U1-Pad11) -> /TMP_VOUT
- U1 pad 12: Net-(U1-Pad12) -> /TMP_nSHDN
- U1 pad 13: Net-(U1-Pad13) -> /AIN_1
- U1 pad 14: Net-(U1-Pad14) -> /BAT_SENSE
- U1 pad 15: Net-(U1-Pad15) -> /AIN_2
- U1 pad 16: Net-(U1-Pad16) -> /THERM
- U1 pad 22: Net-(U1-Pad22) -> /FTU_FIRE
- U1 pad 23: Net-(U1-Pad23) -> /HEAT_ON
- U1 pad 24: Net-(U1-Pad24) -> /uSD_CS
- U1 pad 37: Net-(U1-Pad37) -> /TX
- U1 pad 38: Net-(U1-Pad38) -> /RX
- U1 pad 39: Net-(U1-Pad39) -> /HOST_EN
- U1 pad 41: /HOST_EN -> /MPU_CS
- U1 pad 47: Net-(U1-Pad47) -> /BARO_CS
- U1 pad 48: Net-(U1-Pad48) -> /RADIO_CS
- U1 pad 6: /VDDANA -> 2V5
- U1 pad 7: Net-(U1-Pad7) -> /LED_1
- U1 pad 8: Net-(U1-Pad8) -> /LED_2
- U1 pad 9: Net-(U1-Pad9) -> /LED_3
- U10 pad 2: VIN -> 3V3
- U10 pad 3: VIN -> 3V3
Routing:
- net /HEAT_ON: track 0.00 -> 75.9 mm, vias 0 -> 1
- net /RADIO_CS: track 0.00 -> 68.0 mm, vias 0 -> 2
- net Net-(Q1-Pad1): track 0.00 -> 59.3 mm, vias 0 -> 1
- net /RX: track 0.00 -> 50.6 mm, vias 0 -> 2
- net /RADIO_INT: track 0.00 -> 50.6 mm, vias 0 -> 1
- net /TX: track 0.00 -> 46.1 mm, vias 0 -> 2
- net 2V5: track 0.00 -> 45.9 mm
- net /uSD_CS: track 0.00 -> 33.8 mm, vias 0 -> 2
- net /LED_4: track 0.00 -> 30.8 mm, vias 0 -> 2
- net /LED_3: track 0.00 -> 28.7 mm, vias 0 -> 2
- net /LED_2: track 0.00 -> 27.7 mm, vias 0 -> 2
- net /LED_1: track 0.00 -> 27.5 mm, vias 0 -> 2
- net GND: track 86.4 -> 112.7 mm, vias 60 -> 71
- net /THERM: track 0.00 -> 25.8 mm, vias 0 -> 2
- net Net-(U8-Pad10): track 0.00 -> 22.0 mm
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- added copper zone on F.Cu, net 3V3
- added copper zone on In2.Cu, net 3V3
- added copper zone on In1.Cu, net GND
Other:
- board text added: "A1"
- board text added: "A2"
- board text added: "TMP"

Commit message: Board Done
Connections:
- U1 pad 4: Net-(U1-Pad4) -> /RADIO_INT
Routing:
- net /RADIO_INT: track 50.6 -> 61.5 mm, vias 1 -> 2

Commit message: Changes
Parts:
- removed D4, D5: LED, LEDs:LED_0603
- removed R11: 330, Capacitors_SMD:C_0603
- added J11: Conn_01x02, MASA:A33199CT-ND, F.Cu at (102.5, 121.8)
- added J12: Conn_01x02, MASA:A33199CT-ND, F.Cu at (102.5, 107.2)
- added REF**: Zip_Tie_Hole, MASA:Zip_Tie_Hole, F.Cu at (104.4, 79.6)
- added REF**: Zip_Tie_Hole, MASA:Zip_Tie_Hole, F.Cu at (157.2, 79.6)
- added SW1: SW_Push, Buttons_Switches_SMD:SW_SPST_B3U-1100P, F.Cu at (183.8, 124.6)
- J1: value Conn_02x05_Top_Bottom -> Conn_02x05
- R20: value 330 -> 20k
- R21: value 330 -> 10k
- moved R4 91.4 mm to (102.5, 116.7), turned to 270 degrees
- moved R5 90.3 mm to (102.5, 102.5), turned to 270 degrees
- moved R3 24.6 mm to (182.2, 127.3)
- moved D3 24.6 mm to (179.1, 127.3)
- moved R2 23.5 mm to (182.2, 128.8)
- moved D2 23.5 mm to (179.1, 128.8)
- moved C4 1.13 mm to (179.1, 124.8), turned to 0 degrees
Connections:
- J8 pad 1: GND -> /TX2
- J8 pad 2: /AIN_1 -> /RX2
- J9 pad 2: /AIN_2 -> VIN
- U1 pad 10: /LED_4 -> Net-(U1-Pad10)
- U1 pad 11: /TMP_VOUT -> Net-(U1-Pad11)
- U1 pad 13: /AIN_1 -> Net-(U1-Pad13)
- U1 pad 14: /BAT_SENSE -> Net-(U1-Pad14)
- U1 pad 15: /AIN_2 -> /RX2
- U1 pad 16: /THERM -> /TX2
- U1 pad 19: Net-(U1-Pad19) -> /MOSI
- U1 pad 20: Net-(U1-Pad20) -> /SCLK
- U1 pad 21: Net-(U1-Pad21) -> /MISO
- U1 pad 25: /MOSI -> Net-(U1-Pad25)
- U1 pad 26: /SCLK -> Net-(U1-Pad26)
- U1 pad 27: /MISO -> /LED_4
- U1 pad 28: Net-(U1-Pad28) -> /LED_3
- U1 pad 29: Net-(U1-Pad29) -> /LED_1
- U1 pad 3: Net-(U1-Pad3) -> /RADIO_INT
- U1 pad 30: Net-(U1-Pad30) -> /LED_2
- U1 pad 4: /RADIO_INT -> Net-(U1-Pad4)
- U1 pad 7: /LED_1 -> /TMP_VOUT
- U1 pad 8: /LED_2 -> /BAT_SENSE
- U1 pad 9: /LED_3 -> /THERM
Routing:
- net /LED_4: track 30.8 -> 84.4 mm, vias 2 -> 4
- net /LED_3: track 28.7 -> 78.9 mm, vias 2 -> 4
- net VIN: track 66.8 -> 101.8 mm
- net /TX2: track 0.00 -> 20.6 mm, vias 0 -> 2
- net /LED_2: track 27.7 -> 8.30 mm
- net /HOST_EN: track 18.9 -> 0.00 mm
- net /RX2: track 0.00 -> 17.2 mm, vias 0 -> 2
- net /LED_1: track 27.5 -> 10.6 mm
- net /AIN_1: track 16.2 -> 0.00 mm, vias 2 -> 0
- net /AIN_2: track 15.2 -> 0.00 mm, vias 2 -> 0
- net /MOSI: track 136.9 -> 144.7 mm
- net /SCLK: track 129.1 -> 136.5 mm
- net /MISO: track 125.9 -> 132.5 mm
- net /THERM: track 25.8 -> 31.1 mm
- net /BAT_SENSE: track 12.0 -> 16.7 mm
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Other:
- board text added: "L3"
- board text added: "L4"
- board text added: "TC"
- board text added: "TP"
- board text removed: "A1"
- board text removed: "A2"
- board text removed: "S1"
- board text removed: "S2"
- board text removed: "S3"
- board text removed: "S4"

Commit message: Fixed Stuff
Parts:
- added TP19: TEST, MASA:0603_TP, F.Cu at (170.1, 125.0)
- added TP24: TEST, MASA:0603_TP, F.Cu at (170.6, 127.1)
- moved BT1 1.00 mm to (142.0, 90.0)
- moved BT2 1.00 mm to (119.0, 90.0)
Connections:
- J1 pad 1: /SWDIO -> 3V3
- J1 pad 10: GND -> /nRESET
- J1 pad 2: /SWCLK -> GND
- J1 pad 3: Net-(J1-Pad3) -> GND
- J1 pad 5: /nRESET -> GND
- J1 pad 6: 3V3 -> /SWDIO
- J1 pad 7: GND -> /SWCLK
- J1 pad 8: GND -> Net-(J1-Pad8)
- U1 pad 39: /HOST_EN -> /RADIO_CS
- U1 pad 48: /RADIO_CS -> Net-(U1-Pad48)
Routing:
- net /RADIO_CS: track 68.0 -> 78.4 mm
- net /SWDIO: track 13.9 -> 21.5 mm, vias 0 -> 2
- net /SWCLK: track 15.0 -> 22.5 mm, vias 0 -> 2
- net Net-(TP24-Pad1): track 0.00 -> 5.29 mm
- net /nRESET: track 26.4 -> 31.2 mm
- net Net-(TP19-Pad1): track 0.00 -> 2.35 mm
- net VBAT: track 51.1 -> 52.1 mm
- net GND: track 110.9 -> 110.2 mm
- net /HEAT_ON: track 75.9 -> 76.5 mm
